File: Flightcontrol/kicad/kicad.kicad_pcb (KiCad board)
At the start: 2 copper layers, 60 parts, among them J12 Conn_01x05_Pin, J2 Conn_01x06, J3 Conn_01x08, J4 Conn_01x03_Pin, J5 Conn_01x05, J6 Conn_01x01_Pin, J7 Conn_01x05, U1 ESP32-S3-WROOM-1U-N16R8, U2 BMP581

Commit message: sanity backup
Parts:
- removed J4: Conn_01x03_Pin, Connector_PinHeader_2.54mm:PinHeader_1x03_P2.54mm_Vertical
- removed J6: Conn_01x01_Pin, Connector_PinHeader_2.54mm:PinHeader_1x01_P2.54mm_Vertical
- removed JP1, JP10, JP11, JP14, JP2, JP3, JP8, JP9: SolderJumper_2_Open, Jumper:SolderJumper-2_P1.3mm_Open_RoundedPad1.0x1.5mm
- removed R13, R15: 1.8k, Resistor_SMD:R_0603_1608Metric
- added J1: Conn_01x04_Pin, Connector_PinHeader_2.54mm:PinHeader_1x04_P2.54mm_Vertical, F.Cu at (151.6, 75.1)
- moved J12 141.4 mm to (180.8, 59.9)
- moved J5 138.4 mm to (180.3, 53.5), turned to 90 degrees
- moved J2 85.7 mm to (122.4, 61.6), turned to -90 degrees
- moved RD1 82.6 mm to (132.7, 54.5), turned to 90 degrees
- moved R3 80.8 mm to (133.5, 50.7), turned to -90 degrees
- moved RU1 80.8 mm to (129.4, 54.6), turned to -45 degrees
- moved D1 79.9 mm to (138.7, 51.3), turned to -135 degrees
- moved R9 79.5 mm to (125.4, 73.0), turned to 45 degrees
- moved R2 77.6 mm to (136.3, 50.7), turned to -90 degrees
- moved R16 77.0 mm to (132.0, 72.0), turned to 180 degrees
- moved U2 74.2 mm to (127.4, 69.3), turned to -135 degrees
- moved TP8 72.4 mm to (139.8, 56.9)
- moved R8 71.6 mm to (133.2, 69.4), turned to 90 degrees
- moved C10 71.5 mm to (129.5, 72.4), turned to -90 degrees
- moved C11 69.5 mm to (131.3, 69.5), turned to -90 degrees
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Connections:
- R12 pad 2: Net-(JP8-B) -> /SDA
- R14 pad 2: Net-(JP11-B) -> /SCL
- R9 pad 1: Net-(JP3-A) -> /3.3
- TP1 pad 1: /SDA -> /SCL
- TP2 pad 1: /SCL -> /SDA
- U1 pad 10: /TX -> unconnected-(U1-IO17-Pad10)
- U1 pad 12: /SDA -> /BAR_INT
- U1 pad 17: /SCL -> unconnected-(U1-IO9-Pad17)
- U1 pad 23: unconnected-(U1-IO21-Pad23) -> /GM
- U1 pad 38: unconnected-(U1-IO2-Pad38) -> /RX
- U1 pad 39: unconnected-(U1-IO1-Pad39) -> /TX
- U1 pad 6: /BAR_INT -> unconnected-(U1-IO6-Pad6)
- U1 pad 8: /GM -> /SDA
- U1 pad 9: /RX -> /SCL
Routing:
- net GND: track 0.00 -> 16.4 mm, vias 0 -> 5
- net Net-(J12-Pin_5): track 0.00 -> 10.8 mm
- net /D-: track 0.00 -> 10.7 mm
- net /QM1: track 0.00 -> 10.6 mm
- net Net-(J12-Pin_4): track 0.00 -> 9.78 mm
- net Net-(J12-Pin_3): track 0.00 -> 9.25 mm
- net Net-(J12-Pin_2): track 0.00 -> 8.72 mm
- net Net-(J12-Pin_1): track 0.00 -> 8.20 mm
- net /D+: track 0.00 -> 8.14 mm
- net /GPIO0: track 0.00 -> 5.36 mm
- net /DP: track 0.00 -> 5.19 mm
- net /QM2: track 0.00 -> 4.80 mm
- net /QM3: track 0.00 -> 4.79 mm
- net /QM4: track 0.00 -> 4.78 mm
- net /GM: track 0.00 -> 4.77 mm
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- added copper zone on B.Cu, net GND
Other:
- board text added: "IMU"
- board text added: "MTRS"
- board text added: "PWR"
- board text added: "XCVR"

Commit message: FC.V1 PCB Layout completed
Parts:
- removed J12: Conn_01x05_Pin, Connector_PinHeader_2.54mm:PinHeader_1x05_P2.54mm_Vertical
- removed TP1: x, TestPoint:TestPoint_Pad_D1.5mm
- removed TP2: BAR_CLK, TestPoint:TestPoint_Pad_D1.5mm
- added G***: LOGO, brain:brain, B.Cu at (168.4, 56.4)
- added H1: MountingHole, MountingHole:MountingHole_2.2mm_M2, F.Cu at (131.1, 75.5)
- added H2: MountingHole, MountingHole:MountingHole_2.2mm_M2, F.Cu at (131.1, 46.5)
- added H3: MountingHole, MountingHole:MountingHole_2.2mm_M2, F.Cu at (180.2, 52.3)
- added H4: MountingHole, MountingHole:MountingHole_2.2mm_M2, F.Cu at (180.2, 75.4)
- added J4: Conn_01x01_Pin, Connector_PinHeader_2.54mm:PinHeader_1x01_P2.54mm_Vertical, F.Cu at (133.1, 69.5)
- added J6: Conn_01x03_Pin, Connector_PinHeader_2.54mm:PinHeader_1x03_P2.54mm_Vertical, F.Cu at (181.1, 65.0)
- D1: footprint LED_SMD:LED_0201_0603Metric -> LED_SMD:LED_0603_1608Metric
- TP8: moved to B.Cu
- moved C10 18.3 mm to (146.5, 65.5)
- moved R16 18.3 mm to (149.0, 65.1)
- moved R8 18.3 mm to (150.2, 62.5)
- moved C12 18.3 mm to (152.2, 64.1)
- moved TP4 18.3 mm to (176.2, 72.0)
- moved R9 17.5 mm to (141.5, 66.2), turned to 0 degrees
- moved JP6 16.9 mm to (138.5, 63.1), turned to -90 degrees
- moved C11 16.9 mm to (146.6, 62.3)
- moved U2 16.8 mm to (143.0, 63.0), turned to -90 degrees
- moved JP5 15.9 mm to (137.7, 66.6), turned to -90 degrees
- moved D3 15.4 mm to (175.9, 65.0), turned to 90 degrees
- moved TP8 12.3 mm to (152.1, 57.4)
- moved R10 9.77 mm to (176.3, 68.6), turned to -90 degrees
- moved RD1 9.17 mm to (141.7, 56.3)
- moved J7 9.03 mm to (131.0, 53.6)
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Connections:
- U1 pad 31: Net-(J12-Pin_5) -> /IND_LED
- U1 pad 35: Net-(J12-Pin_1) -> unconnected-(U1-IO42-Pad35)
- U1 pad 41: (no net) -> GND
- U1 pad 5: /IND_LED -> unconnected-(U1-IO5-Pad5)
Routing:
- net /3.3: track 0.00 -> 106.8 mm, vias 0 -> 7
- net GND: track 16.4 -> 59.1 mm, vias 5 -> 17
- net /GPIO0: track 5.36 -> 46.1 mm, vias 0 -> 2
- net /EN: track 4.69 -> 36.4 mm, vias 0 -> 2
- net /SDA: track 0.00 -> 29.5 mm, vias 0 -> 2
- net /SCL: track 0.00 -> 27.1 mm
- net /BATT_A: track 0.00 -> 20.4 mm, vias 0 -> 1
- net /BAR_INT: track 0.00 -> 16.5 mm
- net /QM2: track 4.80 -> 19.5 mm, vias 0 -> 2
- net /QM3: track 4.79 -> 16.9 mm, vias 0 -> 2
- net Net-(J12-Pin_5): track 10.8 -> 0.00 mm
- net Net-(J12-Pin_1): track 8.20 -> 0.00 mm
- net /QM4: track 4.78 -> 12.2 mm, vias 0 -> 2
- net Net-(U2-VDDIO): track 0.00 -> 7.37 mm
- net Net-(JP5-A): track 0.00 -> 6.33 mm
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Other:
- board outline added: 55 x 35.1 mm
- rule pad_to_mask_clearance: 0 -> 0.0508
- board text added: "3.3"
- board text added: "<FLASH"
- board text added: "B"
- board text added: "BAT"
- board text added: "DN"
- board text added: "DP"
- board text added: "E"
- board text added: "FLIGHT CONTROLLER REEF STARNES 11.10.25 V1"
- board text added: "SCL"
- board text added: "⏚"

Commit message: generated pcb files :)
Other:
- board text added: "TX"
Changed lines of the file:
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@@
 		(embedded_fonts no)
 		(model "BMP581.stp"
+			(hide yes)
 			(offset
 				(xyz 0 0 0)
@@
 		)
 		(embedded_fonts no)
-		(model "${KICAD9_3DMODEL_DIR}/RF_Module.3dshapes/ESP32-S3-WROOM-1U.step"
+		(model "${KIPRJMOD}/dependencies/ESP32_S3_WROOM_1U_N16R8/ESP32-S3-WROOM-1U-N16R8.step"
 			(offset
 				(xyz 0 0 0)
@@
 			)
 			(rotate
-				(xyz 0 0 0)
+				(xyz -90 -0 -0)
 			)
 		)
@@
 		(layer "Edge.Cuts")
 	)
+	(gr_text "TX"
+		(at 176.4792 55.4736 90)
+		(layer "F.SilkS")
+		(effects
+			(font
+				(size 1 1)
+				(thickness 0.15)
+			)
+			(justify left bottom)
+		)
+	)
 	(gr_text "BAT"
 		(at 134.5184 54.5592 270)
@@
 			(font
 				(size 1 1)
-				(thickness 0.15)
+				(thickness 0.2)
+				(bold yes)
 				(italic yes)
 			)
@@
 			(font
 				(size 1 1)
-				(thickness 0.15)
+				(thickness 0.2)
+				(bold yes)
 				(italic yes)
 			)
@@
 			(font
 				(size 1 1)
-				(thickness 0.15)
+				(thickness 0.2)
+				(bold yes)
 				(italic yes)
 			)
@@
 	)
 	(gr_text "⏚"
-		(at 134.5184 59.0804 270)
+		(at 134.5692 58.42 270)
 		(layer "F.SilkS")
 		(effects
 			(font
-				(size 1.5 1.5)
-				(thickness 0.1875)
+				(size 1 1)
+				(thickness 0.15)
 			)
 			(justify left bottom)
@@
 		)
 	)
+	(gr_text "⏚"
+		(at 176.6824 61.4172 90)
+		(layer "F.SilkS")
+		(effects
+			(font
+				(size 1 1)
+				(thickness 0.15)
+			)
+			(justify left bottom)
+		)
+	)
 	(gr_text "MTRS"
 		(at 163 72 0)
@@
 			(font
 				(size 1 1)
-				(thickness 0.15)
+				(thickness 0.2)
+				(bold yes)
 				(italic yes)
 			)
@@
 	)
 	(gr_text "IMU"
-		(at 135.9408 60.5536 270)
+		(at 134.5692 59.8424 270)
 		(layer "F.SilkS")
 		(effects
 			(font
 				(size 1 1)
-				(thickness 0.15)
+				(thickness 0.2)
+				(bold yes)
 				(italic yes)
 			)
@@
 	)
 	(zone
+		(net 0)
+		(net_name "")
+		(layer "F.Mask")
+		(hatch edge 0.5)
+		(connect_pads
+			(clearance 0.5)
+		)
+		(min_thickness 0.25)
+		(filled_areas_thickness no)
+		(fill yes
+			(thermal_gap 0.5)
+			(thermal_bridge_width 0.5)
+		)
+		(polygon
+			(pts
+				(xy 141.986 61.976) (xy 141.986 63.9572) (xy 143.9672 63.9572) (xy 143.9672 61.976) (xy 141.9352 61.976)
+				(xy 141.9352 63.9572) (xy 143.9672 63.9572) (xy 143.9672 61.976)
+			)
+		)
+	)
+	(zone
